File: cs.kicad_pcb (KiCad board)
At the start: 2 copper layers, 33 x 14 mm, 12 parts, among them J1 JST_PH4x2mm, U1 APDS-9151, U2 VL53L1CXV0FY_1

Commit message: added led and fixed the apds-9151 not having a connection to vcc
Parts:
- added D1: , LED_SMD:mp1616, F.Cu at (135.8, 88.9)
- added R5: 22R, Resistor_SMD:R_MiniMELF_MMA-0204, F.Cu at (139.9, 88.8)
Connections:
- C1 pad 2: Net-(C1-Pad2) -> +3V3
- C2 pad 2: Net-(C1-Pad2) -> +3V3
- U1 pad 2: Net-(U1-Pad2) -> Net-(R1-Pad2)
- U1 pad 5: Net-(C1-Pad2) -> +3V3
- U1 pad 6: Net-(C1-Pad2) -> +3V3
Routing:
- net +3V3: track 49.2 -> 56.4 mm
- net Net-(C1-Pad2): track 4.09 -> 0.00 mm
- net GND: track 47.4 -> 49.6 mm
- net Net-(D1-Pad2): track 0.00 -> 1.90 mm
Other:
- board text added: ""rev color sensor v3""
- board text removed: "rev color sensor v3 compatible sensor"
